File: cgm_project.kicad_pcb (KiCad board)
At the start: 2 copper layers, 26.2 x 25.3 mm, 37 parts, among them J1 JST BATT CONNECTOR, J2 USB_C_Receptacle_USB2.0_16P, J3 Conn_01x02_MountingPin, Q1 AO3400, SW1 SW_SPDT, SW2 BOOT, SW3 RESET, U1 TP4056-42-ESOP8, U2 AP2112K-3.3, U3 ESP32-C3-WROOM-02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

Commit message: chore: add M2 mounting hole
Parts:
- removed D1: GREEN LED, LED_SMD:LED_0805_2012Metric
- removed D2: RED LED, LED_SMD:LED_0805_2012Metric
- removed SW1: SW_SPDT, Button_Switch_SMD:SW_SPDT_PCM12
- removed SW2: BOOT, Button_Switch_SMD:SW_SPST_B3U-1000P
- removed SW3: RESET, Button_Switch_SMD:SW_SPST_B3U-1000P
- added H1: MountingHole, MountingHole:MountingHole_2.2mm_M2, F.Cu at (174.3, 66.0)
